File: schematics/RackZ80_RS232/RackZ80_RS232.sch (KiCad schematic (older format))
At the start: 18 parts, among them J1 ECB_Kontron, Q1 BC547, U1 74HC245, U2 74LS02, U3 74LS32, U4 74HC245, X1 1.8432MHz

Commit message: Add files via upload
Parts:
- removed unit 4 of U3
- added U11: 74LS08, rackz80_footprints:DIP-14_Socket, symbol 74xx:74LS08
Connections:
- net +5V: now also U11.14 (VCC)
- net GND: now also U11.7 (GND); no longer U2.5, U2.6
- net ~CS: now also U11.1; no longer U1.19 (~CE)
- net ~IntAck: now also U11.2
- net ~RD: no longer U1.1 (A->B)
- net ~WR: now also U1.1 (A->B)
- net ~RESET: now reaches J1.31C (~RESET)
- net ~RESET: now also U2.5, U2.6
- net UART_Controller/RESET: now reaches U2.4
- new net ~BUS: U1.19 (~CE), U11.3
- no-connect marks 39 -> 36
Other:
- note added: "Chip Select & Data Bus"
- note added: "ECB Data Enable.\nEnable when when\nIntAck or CS active."
- note added: "UART Clock & Reset"
- note removed: "Chip Select Logic CS1: 0-7, CS2: 8-F"
- note removed: "UART Clock"
- moved on the sheet: Q1, R1, U2A, U2B, X1
