File: schematics/RackZ80_RS232/logic.sch (KiCad schematic (older format))
At the start: 5 parts, among them SW1 Chip Select, SW2 Vector, U5 74LS138, U6 74HC245

Commit message: Add files via upload
Connections:
- net +5V: now also U6.1 (A->B)
- net GND: no longer U6.1 (A->B)
Changed lines of the file:
@@
 encoding utf-8
 Sheet 2 3
-Title "Project Rack Z80 - RS232"
+Title "Project RackZ80 - RS232"
 Date "2021-04-09"
 Rev "1.0"
@@
 F 3 "" H 4600 5650 50  0001 C CNN
 	1    4600 5650
-	1    0    0    -1
-$EndComp
-$Comp
-L power:GND #PWR022
-U 1 1 609BADC9
-P 5600 5650
-F 0 "#PWR022" H 5600 5400 50  0001 C CNN
-F 1 "GND" H 5605 5477 50  0000 C CNN
-F 2 "" H 5600 5650 50  0001 C CNN
-F 3 "" H 5600 5650 50  0001 C CNN
-	1    5600 5650
 	1    0    0    -1
 $EndComp
@@
 	6000 4150 6000 4200
 Wire Wire Line
-	5600 5300 5600 5650
-Wire Wire Line
 	6000 5500 6000 5650
 $Comp
@@
 Wire Wire Line
 	6400 2600 6450 2600
+Wire Wire Line
+	5600 5300 5450 5300
 Wire Bus Line
 	6700 1000 6700 2500
 Wire Bus Line
 	6700 3500 6700 5100
+Text Label 5450 5300 0    50   ~ 0
++5V
 $EndSCHEMATC
