File: schematics/RackZ80_RS232/uart.sch (KiCad schematic (older format))
At the start: 20 parts, among them J2 Serial 1, J3 Serial 2, U10 MAX232, U7 MAX232, U8 16C550, U9 16C550

Commit message: Add files via upload
Connections:
- net GND: no longer U8.35 (RESET), U9.35 (RESET)
- new net RESET: U8.35 (RESET), U9.35 (RESET)
Changed lines of the file:
@@
 encoding utf-8
 Sheet 3 3
-Title "Project Rack Z80 - RS232"
+Title "Project RackZ80 - RS232"
 Date "2021-04-09"
 Rev "1.0"
@@
 	2250 4150 2250 4200
 Wire Wire Line
-	2850 4200 2850 3950
-Wire Wire Line
 	2850 3550 2750 3550
 $Comp
@@
 Wire Wire Line
 	2750 3750 3150 3750
-Wire Wire Line
-	2750 3950 2850 3950
-Connection ~ 2850 3950
-Wire Wire Line
-	2850 3950 2850 3550
 NoConn ~ 1750 3950
 Wire Wire Line
@@
 	5250 4150 5250 4200
 Wire Wire Line
-	5850 4200 5850 3950
-Wire Wire Line
 	5850 3550 5750 3550
 $Comp
@@
 Wire Wire Line
 	5750 3750 6150 3750
-Wire Wire Line
-	5750 3950 5850 3950
-Connection ~ 5850 3950
-Wire Wire Line
-	5850 3950 5850 3550
 NoConn ~ 4750 3950
 Wire Wire Line
@@
 Wire Wire Line
 	3050 2850 2750 2850
+Wire Wire Line
+	2850 3550 2850 4200
+Text HLabel 3150 3950 2    50   Input ~ 0
+RESET
+Wire Wire Line
+	2750 3950 3150 3950
+Text Label 3050 3950 2    50   ~ 0
+RST
+Wire Wire Line
+	5850 3550 5850 4200
+Wire Wire Line
+	5750 3950 6050 3950
 Wire Bus Line
 	6250 800  6250 3350
@@
 Wire Bus Line
 	6150 650  6150 2250
+Text Label 6050 3950 2    50   ~ 0
+RST
 $EndSCHEMATC
