File: schematics/RackZ80_Backplane/RackZ80_Backplane.kicad_pcb (KiCad board)
At the start: 2 copper layers, 160 x 99 mm, 14 parts, among them J1 ECB_Kontron, J10 -5V, J11 -15V, J12 +15V, J13 PWRCL, J14 GND, J2 ECB_Kontron, J3 ECB_Kontron, J4 ECB_Kontron, J5 ECB_Kontron, J6 ECB_Kontron, J7 ECB_Kontron, J8 ECB_Kontron, J9 +5V

Commit message: migrated kicad 5 to kicad 7
Connections:
- net /~BUSAK renamed /~{BUSAK}
- net /~BUSRQ renamed /~{BUSRQ}
- net /~DPR renamed /~{DPR}
- net /~HLT renamed /~{HLT}
- net /~INT renamed /~{INT}
- net /~IORQ renamed /~{IORQ}
- net /~M1 renamed /~{M1}
- net /~MRQ renamed /~{MRQ}
- net /~NMI renamed /~{NMI}
- net /~PWRCL renamed /~{PWRCL}
- net /~RD renamed /~{RD}
- net /~RESET renamed /~{RESET}
- net /~RFSH renamed /~{RFSH}
- net /~WAIT renamed /~{WAIT}
- net /~WR renamed /~{WR}
- net /~WrEn renamed /~{WrEn}
Other:
- net class Default removed
